File: src/pcb be like.kicad_pcb (KiCad board)
At the start: 2 copper layers, 35 x 56 mm, 21 parts, among them M1 Motor_DC, Q1 2N3906, Q2 2N3906, Q3 2N3904, Q4 2N3904, Q5 2N3904, Q6 2N3904, SW1 SW_Push, SW2 SW_Push

Commit message: final
Parts:
- moved G*** 4.38 mm to (145.0, 79.6)
- moved G*** 1.69 mm to (131.8, 105.0)

Commit message: final final (sent for manufacturing)
Other:
- board text added: "JLCJLCJLCJLC"
- board text removed: "WayWayWay"
Changed lines of the file:
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@@
 		(layer "Edge.Cuts")
 	)
-	(gr_text "WayWayWay"
-		(at 146.65 123.1 0)
+	(gr_text "JLCJLCJLCJLC"
+		(at 146.55 122.9 0)
 		(layer "F.SilkS")
 		(effects
 			(font
-				(size 1 1)
-				(thickness 0.125)
+				(size 1 0.8)
+				(thickness 0.1)
 			)
 			(justify left bottom)
